Commit message: Created script to update udev rules to symlink roomba to /dev/create_2

File: ca_description/urdf/create_base.urdf.xacro (robot description, xacro)
@@ -22,5 +22,5 @@
     </collision>
     </link>
-   <joint name="${prefix}_wheel_joint" type="continuous">
+   <joint name="${prefix}_wheel_joint" type="fixed">
       <origin xyz="0 ${y_offset} 0.015" rpy="0 0 0" />
       <parent link="base_link" />
